Commit message: Fixed URDF file error

File: ros2_ws/src/puzzlebot_description/urdf/puzzlebot.urdf.xacro (robot description, xacro)
@@ -20,8 +20,26 @@
         <origin xyz="0 0 0.05" rpy="0 0 0"/>
     </joint>
+    <!-- Right Wheel -->
+    <link name="wheel_right_link">
+        <visual>
+            <origin xyz="0 0 0" rpy="0 -1.5708 0"/>
+            <geometry>
+                <mesh filename="package://puzzlebot_description/meshes/wheel.stl"/>
+            </geometry>
+            <material name="wheel_color">
+                <color rgba="0.0 0.5 1.0 1.0"/>
+            </material>
+        </visual>
+    </link>
+    <joint name="wheel_right_joint" type="continuous">
+        <parent link="base_link"/>
+        <child link="wheel_right_link"/>
+        <axis xyz="1 0 0"/>
+        <origin xyz="0.098 -0.038 0" rpy="0 0 0"/>
+    </joint>
     <!-- Left Wheel -->
     <link name="wheel_left_link">
         <visual>
-            <origin xyz="0 0 0" rpy="0 -1.5708 0"/>
+            <origin xyz="0 0 0" rpy="0 1.5708 0"/>
             <geometry>
                 <mesh filename="package://puzzlebot_description/meshes/wheel.stl"/>
@@ -36,22 +54,4 @@
         <child link="wheel_left_link"/>
         <axis xyz="1 0 0"/>
-        <origin xyz="0.098 -0.038 0" rpy="0 0 0"/>
-    </joint>
-    <!-- Right Wheel -->
-    <link name="wheel_right_link">
-        <visual>
-            <origin xyz="0 -0.014 0" rpy="0 1.5708 0"/>
-            <geometry>
-                <mesh filename="package://puzzlebot_description/meshes/wheel.stl"/>
-            </geometry>
-            <material name="wheel_color">
-                <color rgba="0.0 0.5 1.0 1.0"/>
-            </material>
-        </visual>
-    </link>
-    <joint name="wheel_right_joint" type="continuous">
-        <parent link="base_link"/>
-        <child link="wheel_right_link"/>
-        <axis xyz="1 0 0"/>
         <origin xyz="-0.098 -0.038 0" rpy="0 0 0"/>
     </joint>

Commit message: Added caster wheel on URDF

File: ros2_ws/src/puzzlebot_description/urdf/puzzlebot.urdf.xacro (robot description, xacro)
@@ -56,3 +56,10 @@
         <origin xyz="-0.098 -0.038 0" rpy="0 0 0"/>
     </joint>
+    <!-- Caster Wheel -->
+    <link name="caster_link"/>
+    <joint name="caster_joint" type="fixed">
+        <parent link="base_footprint"/>
+        <child link="caster_link"/>
+        <origin xyz="0 0.095 0" rpy="0 0 0"/>
+    </joint>
 </robot>

Commit message: Added collision to URDF

File: ros2_ws/src/puzzlebot_description/urdf/puzzlebot.urdf.xacro (robot description, xacro)
@@ -13,4 +13,10 @@
             </material>
         </visual>
+        <collision>
+            <origin xyz="0 0 0" rpy="1.5708 0 0"/>
+            <geometry>
+                <mesh filename="package://puzzlebot_description/meshes/chassis.stl"/>
+            </geometry>
+        </collision>
     </link>
     <!-- Fixed Joint for Base Link -->
@@ -31,4 +37,12 @@
             </material>
         </visual>
+        <collision>
+            <geometry>
+                <origin xyz="0 0 0" rpy="0 0 0"/>
+                <geometry>
+                    <sphere radius="0.05"/>
+                </geometry>
+            </geometry>
+        </collision>
     </link>
     <joint name="wheel_right_joint" type="continuous">
@@ -49,4 +63,12 @@
             </material>
         </visual>
+        <collision>
+            <geometry>
+                <origin xyz="0 0 0" rpy="0 0 0"/>
+                <geometry>
+                    <sphere radius="0.05"/>
+                </geometry>
+            </geometry>
+        </collision>
     </link>
     <joint name="wheel_left_joint" type="continuous">
@@ -57,5 +79,14 @@
     </joint>
     <!-- Caster Wheel -->
-    <link name="caster_link"/>
+    <link name="caster_link">
+        <collision>
+            <geometry>
+                <origin xyz="0 0 0" rpy="0 0 0"/>
+                <geometry>
+                    <sphere radius="0.0075"/>
+                </geometry>
+            </geometry>
+        </collision>
+    </link>
     <joint name="caster_joint" type="fixed">
         <parent link="base_footprint"/>

Commit message: RViz and Gazebo working

File: ros2_ws/src/puzzlebot_description/urdf/puzzlebot.urdf.xacro (robot description, xacro)
@@ -1,8 +1,23 @@
 <?xml version="1.0"?>
 <robot xmlns:xacro="http://ros.org/wiki/xacro" name="puzzlebot">
-    <xacro:include filename="package://puzzlebot_description/urdf/puzzlebot.gazebo.xacro"/>
+    <xacro:include filename="$(find puzzlebot_description)/urdf/puzzlebot_gazebo.xacro"/>
     <!-- Base Links -->
-    <link name="base_footprint"/>
+    <link name="base_footprint">
+        <inertial>
+            <origin xyz="0 0 0" rpy="0 0 0"/>
+            <mass value="0.001"/>
+            <inertia ixx="0.0001" ixy="0.0" ixz="0.0"
+                     iyy="0.0001" iyz="0.0"
+                     izz="0.0001"/>
+        </inertial>
+    </link>
     <link name="base_link">
+        <inertial>
+            <origin xyz="0 0 0" rpy="0 0 0"/>
+            <mass value="0.82573504"/>
+            <inertia ixx="0.001" ixy="0.0" ixz="0.0"
+                     iyy="0.001" iyz="0.0"
+                     izz="0.001"/>
+        </inertial>
         <visual>
             <origin xyz="0 0 0" rpy="1.5708 0 0"/>
@@ -29,4 +44,11 @@
     <!-- Right Wheel -->
     <link name="wheel_right_link">
+        <inertial>
+            <origin xyz="0 0 0" rpy="0 0 0"/>
+            <mass value="0.053"/>
+            <inertia ixx="0.001" ixy="0.0" ixz="0.0"
+                     iyy="0.001" iyz="0.0"
+                     izz="0.001"/>
+        </inertial>
         <visual>
             <origin xyz="0 0 0" rpy="0 -1.5708 0"/>
@@ -39,9 +61,7 @@
         </visual>
         <collision>
+            <origin xyz="0 0 0" rpy="0 0 0"/>
             <geometry>
-                <origin xyz="0 0 0" rpy="0 0 0"/>
-                <geometry>
-                    <sphere radius="0.05"/>
-                </geometry>
+                <sphere radius="0.05"/>
             </geometry>
         </collision>
@@ -55,4 +75,11 @@
     <!-- Left Wheel -->
     <link name="wheel_left_link">
+        <inertial>
+            <origin xyz="0 0 0" rpy="0 0 0"/>
+            <mass value="0.053"/>
+            <inertia ixx="0.001" ixy="0.0" ixz="0.0"
+                     iyy="0.001" iyz="0.0"
+                     izz="0.001"/>
+        </inertial>
         <visual>
             <origin xyz="0 0 0" rpy="0 1.5708 0"/>
@@ -65,9 +92,7 @@
         </visual>
         <collision>
+            <origin xyz="0 0 0" rpy="0 0 0"/>
             <geometry>
-                <origin xyz="0 0 0" rpy="0 0 0"/>
-                <geometry>
-                    <sphere radius="0.05"/>
-                </geometry>
+                <sphere radius="0.05"/>
             </geometry>
         </collision>
@@ -81,10 +106,15 @@
     <!-- Caster Wheel -->
     <link name="caster_link">
+        <inertial>
+            <origin xyz="0 0 0" rpy="0 0 0"/>
+            <mass value="1.44379265037903E-06"/>
+            <inertia ixx="1.0E-10" ixy="0.0" ixz="0.0"
+                     iyy="1.0E-10" iyz="0.0"
+                     izz="1.0E-10"/>
+        </inertial>
         <collision>
+            <origin xyz="0 0 0" rpy="0 0 0"/>
             <geometry>
-                <origin xyz="0 0 0" rpy="0 0 0"/>
-                <geometry>
-                    <sphere radius="0.0075"/>
-                </geometry>
+                <sphere radius="0.0075"/>
             </geometry>
         </collision>

Commit message: Added bringup package and tested teleop with Xbox

File: ros2_ws/src/puzzlebot_description/urdf/puzzlebot.urdf.xacro (robot description, xacro)
@@ -17,5 +17,5 @@
         <inertial>
             <origin xyz="0 0 0" rpy="0 0 0"/>
-            <mass value="0.82573504"/>
+            <mass value="1.2"/>
             <inertia ixx="0.001" ixy="0.0" ixz="0.0"
                      iyy="0.001" iyz="0.0"
